Commit message: 建立 UGV-UAV 协同配送仿真 v1.0.0 基线

File: wqi_final/simulation_ws/src/ugvcar_description/urdf/ugvcar/base.urdf.xacro (robot description, xacro)
@@ -10,5 +10,5 @@
         </joint>
         <link name="base_link">
-            <visual>
+            <visual name="chassis_visual">
                 <origin xyz="0 0 0.0" rpy="0 0 0" />
                 <geometry>
@@ -16,5 +16,24 @@
                 </geometry>
                 <material name="blue">
-                    <color rgba="0.1 0.1 1.0 0.5"/>
+                    <color rgba="0.1 0.25 0.9 1.0"/>
+                </material>
+            </visual>
+            <!-- Visual-only carrier deck keeps the validated collision footprint unchanged. -->
+            <visual name="carrier_support_visual">
+                <origin xyz="0 0 0.175" rpy="0 0 0" />
+                <geometry>
+                    <box size="0.18 0.14 0.23" />
+                </geometry>
+                <material name="carrier_dark">
+                    <color rgba="0.12 0.15 0.18 1.0"/>
+                </material>
+            </visual>
+            <visual name="uav_docking_deck_visual">
+                <origin xyz="0 0 0.309" rpy="0 0 0" />
+                <geometry>
+                    <box size="0.62 0.50 0.04" />
+                </geometry>
+                <material name="carrier_orange">
+                    <color rgba="0.95 0.42 0.05 1.0"/>
                 </material>
             </visual>

File: wqi_final/simulation_ws/src/ugvcar_description/urdf/ugvcar/plugins/gazebo_sensor_plugin.xacro (robot description, xacro)
@@ -13,5 +13,5 @@
                 </plugin>
                 <always_on>true</always_on>
-                <visualize>true</visualize>
+                <visualize>$(arg visualize_sensor_rays)</visualize>
                 <update_rate>10</update_rate>
                 <pose>0 0 0 0 0 0</pose>

File: wqi_final/simulation_ws/src/ugvcar_description/urdf/ugvcar/ugvcar.ros2_control.xacro (robot description, xacro)
@@ -8,6 +8,6 @@
             <joint name="left_wheel_joint">
                 <command_interface name="velocity">
-                    <param name="min">-1</param>
-                    <param name="max">1</param>
+                    <param name="min">-40</param>
+                    <param name="max">40</param>
                 </command_interface>
                 <command_interface name="effort">
@@ -21,6 +21,6 @@
             <joint name="right_wheel_joint">
                 <command_interface name="velocity">
-                    <param name="min">-1</param>
-                    <param name="max">1</param>
+                    <param name="min">-40</param>
+                    <param name="max">40</param>
                 </command_interface>
                 <command_interface name="effort">

File: wqi_final/simulation_ws/src/ugvcar_description/urdf/ugvcar/ugvcar.urdf.xacro (robot description, xacro)
@@ -1,4 +1,5 @@
 <?xml version="1.0"?>
 <robot xmlns:xacro="http://www.ros.org/wiki/xacro" name="ugvcar">
+    <xacro:arg name="visualize_sensor_rays" default="false" />
     <xacro:include filename="$(find ugvcar_description)/urdf/ugvcar/base.urdf.xacro" />
     <!-- 传感器组件 -->
@@ -26,3 +27,16 @@
     <xacro:include filename="$(find ugvcar_description)/urdf/ugvcar/plugins/gazebo_sensor_plugin.xacro" />
     <xacro:gazebo_sensor_plugin />
+    <!-- Simulation ground truth used to keep map/RViz aligned with Gazebo. -->
+    <gazebo>
+        <plugin name="ugvcar_ground_truth" filename="libgazebo_ros_p3d.so">
+            <ros>
+                <namespace>/</namespace>
+                <remapping>odom:=ground_truth/odom</remapping>
+            </ros>
+            <body_name>base_footprint</body_name>
+            <frame_name>world</frame_name>
+            <update_rate>50.0</update_rate>
+            <gaussian_noise>0.0</gaussian_noise>
+        </plugin>
+    </gazebo>
 </robot>
