Commit message: 更新 PX4 四车分区协同配送与导航修复基线
纳入固定版本 PX4 子模块、分区校园和四车部署，保留已确认的旧 UI 与替代飞控移除。修复返站转角规划净空和 Offboard 健康检查时间竞态，更新测试与中文文档。完整食堂二楼配送功能通过；RViz 关闭异常仍作为已知问题记录。

File: wqi_final/simulation_ws/src/uav_description/urdf/uav.urdf.xacro (robot description, xacro)
@@ -65,5 +65,5 @@
     <inertial>
       <origin xyz="0 0 0.15" rpy="0 0 0"/>
-      <mass value="1.477"/>
+      <mass value="1.535"/>
       <inertia ixx="0.1152" ixy="0" ixz="0" iyy="0.1152" iyz="0" izz="0.218"/>
     </inertial>
@@ -194,38 +194,4 @@
   </gazebo>
   <gazebo>
-    <plugin name="campus_uav_dynamics" filename="libplugin_drone.so">
-      <ros><namespace>${model['namespace']}</namespace></ros>
-      <bodyName>base_link</bodyName>
-      <pub_odom>true</pub_odom>
-      <odom_hz>30</odom_hz>
-      <rollpitchProportionalGain>${model['rollpitchProportionalGain']}</rollpitchProportionalGain>
-      <rollpitchDifferentialGain>${model['rollpitchDifferentialGain']}</rollpitchDifferentialGain>
-      <rollpitchLimit>${model['rollpitchLimit']}</rollpitchLimit>
-      <yawProportionalGain>${model['yawProportionalGain']}</yawProportionalGain>
-      <yawDifferentialGain>${model['yawDifferentialGain']}</yawDifferentialGain>
-      <yawLimit>${model['yawLimit']}</yawLimit>
-      <velocityXYProportionalGain>${model['velocityXYProportionalGain']}</velocityXYProportionalGain>
-      <velocityXYDifferentialGain>${model['velocityXYDifferentialGain']}</velocityXYDifferentialGain>
-      <velocityXYLimit>${model['velocityXYLimit']}</velocityXYLimit>
-      <velocityZProportionalGain>${model['velocityZProportionalGain']}</velocityZProportionalGain>
-      <velocityZIntegralGain>${model['velocityZIntegralGain']}</velocityZIntegralGain>
-      <velocityZDifferentialGain>${model['velocityZDifferentialGain']}</velocityZDifferentialGain>
-      <velocityZLimit>${model['velocityZLimit']}</velocityZLimit>
-      <positionXYProportionalGain>${model['positionXYProportionalGain']}</positionXYProportionalGain>
-      <positionXYDifferentialGain>${model['positionXYDifferentialGain']}</positionXYDifferentialGain>
-      <positionXYIntegralGain>${model['positionXYIntegralGain']}</positionXYIntegralGain>
-      <positionXYLimit>${model['positionXYLimit']}</positionXYLimit>
-      <positionZProportionalGain>${model['positionZProportionalGain']}</positionZProportionalGain>
-      <positionZDifferentialGain>${model['positionZDifferentialGain']}</positionZDifferentialGain>
-      <positionZIntegralGain>${model['positionZIntegralGain']}</positionZIntegralGain>
-      <positionZLimit>${model['positionZLimit']}</positionZLimit>
-      <maxForce>${model['maxForce']}</maxForce>
-      <motionSmallNoise>${model['motionSmallNoise']}</motionSmallNoise>
-      <motionDriftNoise>${model['motionDriftNoise']}</motionDriftNoise>
-      <motionDriftNoiseTime>${model['motionDriftNoiseTime']}</motionDriftNoiseTime>
-      <landingVelocity>${model['landingVelocity']}</landingVelocity>
-      <landingHeight>${model['landingHeight']}</landingHeight>
-      <landingTolerance>${model['landingTolerance']}</landingTolerance>
-    </plugin>
     <xacro:if value="$(arg enable_docking)">
       <plugin name="ugv_uav_docking" filename="libugv_uav_docking_plugin.so">
